File: CI_ComPCB/CI_ComPCB.kicad_pcb (KiCad board)
At the start: 2 copper layers, 78.7 x 66 mm, 26 parts, among them IC201 TPS54331DR, J101 Conn_01x01_Male, J201 Connector_Conn_01x01_Male, J202 Conn_01x01_Male, J301 RJ45_LED_Shielded, U101 ESP32s

Commit message: prilim pcb finished
Parts:
- added F201: MF-MSMF050-2, SamacSys_Parts:FUSC4632X85N, F.Cu at (123.5, 70.5)
- added R302: 680, Resistor_SMD:R_0805_2012Metric, F.Cu at (137.8, 90.5)
- added RT201: SL08_10001, SamacSys_Parts:SL0810001, F.Cu at (124.5, 74.7)
- added U102: oled(128x64)i2c, CI_ComPCB:oled(128x64)i2c, B.Cu at (151.4, 81.7)
- moved R301 18.8 mm to (135.5, 90.5)
- moved J201 8.11 mm to (137.3, 117.1)
- moved C201 0.64 mm to (132.9, 119.5)
- moved C204 0.64 mm to (137.8, 110.5)
- moved IC201 0.64 mm to (133.7, 109.6)
- moved R201 0.64 mm to (129.5, 96.9)
- moved L201 0.64 mm to (123.0, 98.7)
- moved C208 0.64 mm to (121.1, 108.1)
- moved D201 0.64 mm to (126.6, 110.1)
- moved D202 0.64 mm to (122.5, 117.7)
- moved C202 0.64 mm to (133.0, 115.7)
- moved C203 0.64 mm to (129.6, 105.0)
- moved C206 0.64 mm to (121.0, 112.9)
- moved C207 0.64 mm to (129.6, 100.5)
- moved J202 0.64 mm to (128.1, 118.2)
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Connections:
- C201 pad 1: EPower -> Net-(C201-Pad1)
- C202 pad 1: EPower -> Net-(C201-Pad1)
- IC201 pad 2: EPower -> Net-(C201-Pad1)
- IC201 pad 3: Net-(IC201-Pad3) -> (no net)
- J201 pad 1: EPower -> Net-(C201-Pad1)
- J301 pad 11: Net-(J301-Pad11) -> GND
- J301 pad 3: Net-(J301-Pad3) -> (no net)
- J301 pad 4: Net-(J301-Pad4) -> (no net)
- J301 pad 5: Net-(J301-Pad5) -> (no net)
- J301 pad 6: Net-(J301-Pad6) -> (no net)
- R301 pad 1: Net-(J301-Pad10) -> RX2
- R301 pad 2: EPower -> Net-(J301-Pad10)
- U101 pad D12: Net-(U101-PadD12) -> (no net)
- U101 pad D13: Net-(U101-PadD13) -> (no net)
- U101 pad D14: Net-(U101-PadD14) -> (no net)
- U101 pad D15: Net-(U101-PadD15) -> (no net)
- U101 pad D18: Net-(U101-PadD18) -> (no net)
- U101 pad D19: Net-(U101-PadD19) -> (no net)
- U101 pad D2: Net-(U101-PadD2) -> (no net)
- U101 pad D23: Net-(U101-PadD23) -> (no net)
- U101 pad D25: Net-(U101-PadD25) -> (no net)
- U101 pad D26: Net-(U101-PadD26) -> (no net)
- U101 pad D27: Net-(U101-PadD27) -> (no net)
- U101 pad D32: Net-(U101-PadD32) -> (no net)
- U101 pad D33: Net-(U101-PadD33) -> (no net)
- U101 pad D34: Net-(U101-PadD34) -> (no net)
- U101 pad D35: Net-(U101-PadD35) -> (no net)
- U101 pad D4: Net-(U101-PadD4) -> (no net)
- U101 pad D5: Net-(U101-PadD5) -> (no net)
- U101 pad EN: Net-(U101-PadEN) -> (no net)
- U101 pad RX0: Net-(U101-PadRX0) -> (no net)
- U101 pad TX0: Net-(U101-PadTX0) -> (no net)
- U101 pad VN: Net-(U101-PadVN) -> (no net)
- U101 pad VP: Net-(U101-PadVP) -> (no net)
Routing:
- net EPower: track 93.5 -> 17.0 mm
- net Net-(C201-Pad1): track 0.00 -> 55.6 mm
- net 3.3V: track 10.5 -> 58.2 mm, vias 0 -> 3
- net Net-(U101-PadD21): track 0.00 -> 28.4 mm
- net RX2: track 20.8 -> 48.0 mm
- net Net-(J301-Pad12): track 0.00 -> 24.0 mm
- net TX2: track 22.8 -> 44.3 mm, vias 2 -> 1
- net GND: track 99.3 -> 79.3 mm, vias 25 -> 23
- net B1: track 31.3 -> 47.2 mm
- net Net-(U101-PadD22): track 0.00 -> 11.2 mm
- net Net-(F201-Pad2): track 0.00 -> 5.56 mm
- net Net-(J301-Pad10): track 8.69 -> 14.0 mm
- net A1: track 21.3 -> 25.6 mm
Other:
- board text added: "Innovive Jan 2022 V1.3b_production"
- board text removed: "Innovive Jan 2022 V1.2b_production"

Commit message: temp2
Parts:
- C201, C202: footprint Capacitor_SMD:C_1210_3225Metric -> Capacitor_SMD:C_1206_3216Metric
- C206, C208: footprint Capacitor_SMD:C_1210_3225Metric -> Capacitor_SMD:C_0805_2012Metric
- moved C203 2.75 mm to (127.1, 104.0), turned to 0 degrees
- moved U102 2.50 mm to (151.4, 84.2)
- moved C205 2.13 mm to (133.1, 99.6)
- moved IC201 2.03 mm to (131.8, 109.0)
- moved C204 2.03 mm to (135.8, 109.9)
- moved R202 1.26 mm to (133.2, 95.6)
- moved C206 0.84 mm to (120.7, 112.1)
- moved R301 0.56 mm to (135.6, 91.1)
- moved R302 0.54 mm to (137.8, 91.1)
- moved C202 0.29 mm to (132.9, 116.0)
- moved C208 0.28 mm to (120.8, 108.2)
- moved C201 0.17 mm to (132.9, 119.3)
Routing:
- net Net-(C206-Pad1): track 41.4 -> 36.8 mm
- net Net-(C205-Pad2): track 7.17 -> 3.42 mm
- net Net-(U101-PadD22): track 11.2 -> 8.88 mm
- net Net-(U101-PadD21): track 28.4 -> 26.4 mm
- net Net-(J301-Pad12): track 24.0 -> 25.4 mm
- net Net-(C203-Pad2): track 7.28 -> 8.41 mm
- net 3.3V: track 58.2 -> 57.1 mm
- net RX2: track 48.0 -> 47.2 mm
- net Net-(J301-Pad10): track 14.0 -> 14.7 mm
- net Net-(IC201-Pad5): track 16.5 -> 15.9 mm
- net Vin: track 13.5 -> 12.9 mm
Other:
- board text added: "3.3v"
- board text added: "RX"
- board text added: "SCL"
- board text added: "SDA"
- board text added: "TX"
- board text added: "Vout"
- board text removed: "Vout Diss"

Commit message: print
Parts:
- R201: value 56.2k -> 56k
- R202: value 10.2k -> 10k
- R203: value 1.78k -> 1.8k
Changed lines of the file:
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@@
     (mod_text_size 1 1)
     (mod_text_width 0.15)
-    (pad_size 1.5 3.43)
-    (pad_drill 0)
+    (pad_size 3.25 3.25)
+    (pad_drill 3.25)
     (pad_to_mask_clearance 0)
     (aux_axis_origin 65 163)
@@
     (add_net "Net-(C206-Pad1)")
     (add_net "Net-(F201-Pad2)")
-    (add_net "Net-(IC201-Pad3)")
     (add_net "Net-(IC201-Pad5)")
     (add_net "Net-(J301-Pad10)")
     (add_net "Net-(J301-Pad12)")
-    (add_net "Net-(J301-Pad3)")
-    (add_net "Net-(J301-Pad4)")
-    (add_net "Net-(J301-Pad5)")
-    (add_net "Net-(J301-Pad6)")
-    (add_net "Net-(U101-PadD12)")
-    (add_net "Net-(U101-PadD13)")
-    (add_net "Net-(U101-PadD14)")
-    (add_net "Net-(U101-PadD15)")
-    (add_net "Net-(U101-PadD18)")
-    (add_net "Net-(U101-PadD19)")
-    (add_net "Net-(U101-PadD2)")
     (add_net "Net-(U101-PadD21)")
     (add_net "Net-(U101-PadD22)")
-    (add_net "Net-(U101-PadD23)")
-    (add_net "Net-(U101-PadD25)")
-    (add_net "Net-(U101-PadD26)")
-    (add_net "Net-(U101-PadD27)")
-    (add_net "Net-(U101-PadD32)")
-    (add_net "Net-(U101-PadD33)")
-    (add_net "Net-(U101-PadD34)")
-    (add_net "Net-(U101-PadD35)")
-    (add_net "Net-(U101-PadD4)")
-    (add_net "Net-(U101-PadD5)")
-    (add_net "Net-(U101-PadEN)")
-    (add_net "Net-(U101-PadRX0)")
-    (add_net "Net-(U101-PadTX0)")
-    (add_net "Net-(U101-PadVN)")
-    (add_net "Net-(U101-PadVP)")
     (add_net RX2)
     (add_net TX2)
@@
     (fp_text value 22uf (at 0 1.85) (layer F.Fab)
       (effects (font (size 1 1) (thickness 0.15)))
-    )
-    (fp_text user %R (at 0 0) (layer F.Fab)
-      (effects (font (size 0.8 0.8) (thickness 0.12)))
     )
     (fp_line (start -1.6 0.8) (end -1.6 -0.8) (layer F.Fab) (width 0.1))
@@
     (fp_line (start 2.3 -1.15) (end 2.3 1.15) (layer F.CrtYd) (width 0.05))
     (fp_line (start 2.3 1.15) (end -2.3 1.15) (layer F.CrtYd) (width 0.05))
+    (fp_text user %R (at 0 0) (layer F.Fab)
+      (effects (font (size 0.8 0.8) (thickness 0.12)))
+    )
     (pad 2 smd roundrect (at 1.475 0 180) (size 1.15 1.8) (layers F.Cu F.Paste F.Mask) (roundrect_rratio 0.217391)
       (net 1 GND))
@@
     (fp_text value 22uf (at 0 1.85) (layer F.Fab)
       (effects (font (size 1 1) (thickness 0.15)))
-    )
-    (fp_text user %R (at 0 0) (layer F.Fab)
-      (effects (font (size 0.8 0.8) (thickness 0.12)))
     )
     (fp_line (start -1.6 0.8) (end -1.6 -0.8) (layer F.Fab) (width 0.1))
@@
     (fp_line (start 2.3 -1.15) (end 2.3 1.15) (layer F.CrtYd) (width 0.05))
     (fp_line (start 2.3 1.15) (end -2.3 1.15) (layer F.CrtYd) (width 0.05))
+    (fp_text user %R (at 0 0) (layer F.Fab)
+      (effects (font (size 0.8 0.8) (thickness 0.12)))
+    )
     (pad 2 smd roundrect (at 1.475 0 180) (size 1.15 1.8) (layers F.Cu F.Paste F.Mask) (roundrect_rratio 0.217391)
       (net 1 GND))
@@
     (fp_text value 47uF (at 0 1.68) (layer F.Fab)
       (effects (font (size 1 1) (thickness 0.15)))
-    )
-    (fp_text user %R (at 0 0) (layer F.Fab)
-      (effects (font (size 0.5 0.5) (thickness 0.08)))
     )
     (fp_line (start -1 0.625) (end -1 -0.625) (layer F.Fab) (width 0.1))
@@
     (fp_line (start 1.7 -0.98) (end 1.7 0.98) (layer F.CrtYd) (width 0.05))
     (fp_line (start 1.7 0.98) (end -1.7 0.98) (layer F.CrtYd) (width 0.05))
+    (fp_text user %R (at 0 0) (layer F.Fab)
+      (effects (font (size 0.5 0.5) (thickness 0.08)))
+    )
     (pad 2 smd roundrect (at 0.95 0) (size 1 1.45) (layers F.Cu F.Paste F.Mask) (roundrect_rratio 0.25)
       (net 1 GND))
@@
     (fp_text value 47uF (at 0 1.68) (layer F.Fab)
       (effects (font (size 1 1) (thickness 0.15)))
-    )
-    (fp_text user %R (at 0 0) (layer F.Fab)
-      (effects (font (size 0.5 0.5) (thickness 0.08)))
     )
     (fp_line (start -1 0.625) (end -1 -0.625) (layer F.Fab) (width 0.1))
@@
     (fp_line (start 1.7 -0.98) (end 1.7 0.98) (layer F.CrtYd) (width 0.05))
     (fp_line (start 1.7 0.98) (end -1.7 0.98) (layer F.CrtYd) (width 0.05))
+    (fp_text user %R (at 0 0) (layer F.Fab)
+      (effects (font (size 0.5 0.5) (thickness 0.08)))
+    )
     (pad 2 smd roundrect (at 0.95 0) (size 1 1.45) (layers F.Cu F.Paste F.Mask) (roundrect_rratio 0.25)
       (net 1 GND))
@@
   (module CI_ComPCB:TXRX-AB (layer F.Cu)
     (at 148.82 128.075 90)
+    (attr smd)
     (fp_text reference Converter301 (at 1 -1 90) (layer F.SilkS)
       (effects (font (size 1 1) (thickness 0.15)))
@@
       (effects (font (size 1 1) (thickness 0.15)))
     )
-    (fp_text value 1.78k (at 0 1.65) (layer F.Fab)
+    (fp_text value 1.8k (at 0 1.65) (layer F.Fab)
       (effects (font (size 1 1) (thickness 0.15)))
     )
@@
       (effects (font (size 1 1) (thickness 0.15)))
     )
-    (fp_text value 10.2k (at 0 1.65 90) (layer F.Fab)
+    (fp_text value 10k (at 0 1.65 90) (layer F.Fab)
       (effects (font (size 1 1) (thickness 0.15)))
     )
@@
       (effects (font (size 1 1) (thickness 0.15)))
     )
-    (fp_text value 56.2k (at 0 1.65) (layer F.Fab)
-      (effects (font (size 1 1) (thickness 0.15)))
-    )
+    (fp_text value 56k (at 0 1.65) (layer F.Fab)
+      (effects (font (size 1 1) (thickness 0.15)))
+    )
