File: CI_ComPCB/CI_ComPCB.sch (KiCad schematic (older format))
At the start: 30 parts, among them J1 Conn_01x15_Female, J10 Conn_01x02_Male, J1001 Conn_01x06_Female, J1002 Conn_01x06_Female, J1003 Conn_02x04_Odd_Even, J11 Conn_01x02_Male, J12 Conn_01x01_Female, J13 Conn_01x01_Female, J2 Conn_01x02_Male, J4 Conn_01x15_Female, J6 Conn_01x02_Male, J7 Conn_01x03_Male, J8 RJ45_LED_Shielded, J9 RJ45_LED_Shielded, Q1 IRF9540N, Q2 IRF9540N, U1 Boost_Converter, U1001 ESP32s

Commit message: Rough V1
Parts:
- removed Buck_Converter1: 12v_to_5V, RackCom:12vto5v, symbol CI_ComPCB-rescue:12v_to_5V-New_Library-RackComm-rescue
- removed D1, D2, D3: 1N5400, Diode_THT:D_DO-201AD_P15.24mm_Horizontal, symbol Diode:1N5400
- removed HW-3731: Charger, RackCom:Charger, symbol CI_ComPCB-rescue:Charger-New_Library-RackComm-rescue-RackComm-rescue
- removed Holder1: Battery-New_Library, RackCom:Battery, symbol CI_ComPCB-rescue:Battery-New_Library-RackComm-rescue
- removed J10, J2, J6: Conn_01x02_Male, Connector_PinHeader_2.54mm:PinHeader_1x02_P2.54mm_Vertical, symbol Connector:Conn_01x02_Male
- removed J7: Conn_01x03_Male, Connector_PinHeader_2.54mm:PinHeader_1x03_P2.54mm_Vertical, symbol Connector:Conn_01x03_Male
- removed Q2: IRF9540N, Package_TO_SOT_THT:TO-220-3_Vertical, symbol Transistor_FET:IRF9540N
- removed U1: Boost_Converter, RackCom:BoostConverter, symbol CI_ComPCB-rescue:Boost_Converter-New_Library-RackComm-rescue
- added C1001, C1004: 4700pF, Capacitor_SMD:C_0805_2012Metric, symbol Device:C
- added C1002: 0.1uF, Capacitor_SMD:C_0805_2012Metric, symbol Device:C
- added C1003: 0.01uF, Capacitor_SMD:C_0805_2012Metric, symbol Device:C
- added C1005, C1007: 33uF, Capacitor_SMD:C_0805_2012Metric, symbol Device:C
- added C1006: 39pF, Capacitor_SMD:C_0805_2012Metric, symbol Device:C
- added D1001, D1003: 1N5400, Diode_THT:D_DO-201AD_P12.70mm_Horizontal, symbol Diode:1N5400
- added D1002: B340A-13-F, digikey-footprints:DO-214AC, symbol dk_Diodes-Rectifiers-Single:B340A-13-F
- added J1001, J1007, J1008: Conn_01x02_Male, Connector_PinHeader_2.54mm:PinHeader_1x02_P2.54mm_Vertical, symbol Connector:Conn_01x02_Male
- added L1001: 6.8uH, digikey-footprints:Inductor_13R106C, symbol Device:L_Core_Iron
- added R1001: 332k, Resistor_SMD:R_0805_2012Metric, symbol Device:R
- added R1002: 68.1k, Resistor_SMD:R_0805_2012Metric, symbol Device:R
- added R1003: 44.9K, Resistor_SMD:R_0805_2012Metric, symbol Device:R
- added R1004: 10k, Resistor_SMD:R_0805_2012Metric, symbol Device:R
- added R1005: 1.91k, Resistor_SMD:R_0805_2012Metric, symbol Device:R
- added U1002: TPS54331, Package_SO:TI_SO-PowerPAD-8, symbol CI_ComPCB-rescue:TPS54331
- Converter1001: renamed from Converter2; footprint RackCom:TXRX-AB -> CI_ComPCB:TXRX-AB
- Converter1002: renamed from Converter1; footprint RackCom:TXRX-AB -> CI_ComPCB:TXRX-AB
- J1011: renamed from J12; footprint Connector_PinSocket_2.54mm:PinSocket_1x01_P2.54mm_Vertical -> Connector_PinHeader_2.54mm:PinHeader_1x01_P2.54mm_Vertical
- J1012: renamed from J13; footprint Connector_PinSocket_2.54mm:PinSocket_1x01_P2.54mm_Vertical -> Connector_PinHeader_2.54mm:PinHeader_1x01_P2.54mm_Vertical
- J1013: renamed from J1003; footprint Connector_PinHeader_2.00mm:PinHeader_2x04_P2.00mm_Vertical -> Connector_PinHeader_2.54mm:PinHeader_2x04_P2.54mm_Vertical
- Q1001: renamed from Q1; footprint Package_TO_SOT_THT:TO-220-3_Vertical -> digikey-footprints:TO-220-3
- R1006: renamed from R1; footprint Resistor_SMD:R_2512_6332Metric_Pad1.52x3.35mm_HandSolder -> Resistor_SMD:R_0805_2012Metric
- R1007: renamed from R2; footprint Resistor_SMD:R_2512_6332Metric_Pad1.52x3.35mm_HandSolder -> Resistor_SMD:R_0805_2012Metric
- R1008: renamed from R3; footprint Resistor_SMD:R_2512_6332Metric_Pad1.52x3.35mm_HandSolder -> Resistor_SMD:R_0805_2012Metric
- R1009: renamed from R4; footprint Resistor_SMD:R_2512_6332Metric_Pad1.52x3.35mm_HandSolder -> Resistor_SMD:R_0805_2012Metric
- U1001: footprint RackCom:ESP32s -> CI_ComPCB:ESP32s
- renumbered J11 to J1002, J1 to J1003, J4 to J1004, J1001 to J1005, J1002 to J1006, J8 to J1009, J9 to J1010
Connections:
- wire segments 145 -> 178
Other:
- note added: "R1001 and 1002 need to be changed to be a voltage divider\n"

Commit message: V1 w/ no Battery
Parts:
- removed J1007: Conn_01x02_Male, Connector_PinHeader_2.54mm:PinHeader_1x02_P2.54mm_Vertical, symbol Connector:Conn_01x02_Male
- removed L1001: 6.8uH, digikey-footprints:Inductor_13R106C, symbol Device:L_Core_Iron
- removed R1002: 68.1k, Resistor_SMD:R_0805_2012Metric, symbol Device:R
- added C1008: 10uF, Capacitor_SMD:C_0805_2012Metric, symbol Device:C
- added L1001: SRN8040-100M, SamacSys_Parts:SRN8040100M, symbol SamacSys_Parts:SRN8040-100M
- C1001: value 4700pF -> 10uF
- C1002: value 0.1uF -> 100nF
- C1003: value 0.01uF -> 8.2nF
- C1004: value 4700pF -> 1nF
- C1005, C1007: value 33uF -> 47uF
- C1006: value 39pF -> 10pf
- R1001: value 332k -> 0
- R1003: value 44.9K -> 49.9k
- R1004: value 10k -> 10.2k
Connections:
- wire segments 178 -> 169
Other:
- note removed: "R1001 and 1002 need to be changed to be a voltage divider\n"
Changed lines of the file:
@@
 F 3 "http://www.irf.com/product-info/datasheets/data/irf9540n.pdf" H 1500 1700 50  0001 L CNN
 	1    1500 1700
-	0    -1   1    0
+	0    1    1    0
 $EndComp
 $Comp
@@
 Connection ~ 4850 1000
 $Comp
-L Device:L_Core_Iron L1001
-U 1 1 61242DE6
-P 5450 1000
-F 0 "L1001" V 5675 1000 50  0000 C CNN
-F 1 "6.8uH" V 5584 1000 50  0000 C CNN
-F 2 "digikey-footprints:Inductor_13R106C" H 5450 1000 50  0001 C CNN
-F 3 "~" H 5450 1000 50  0001 C CNN
-	1    5450 1000
-	0    -1   -1   0
-$EndComp
-$Comp
 L Device:C C1005
 U 1 1 6124A796
 P 5700 1400
 F 0 "C1005" H 5815 1446 50  0000 L CNN
-F 1 "33uF" H 5815 1355 50  0000 L CNN
+F 1 "47uF" H 5815 1355 50  0000 L CNN
 F 2 "Capacitor_SMD:C_0805_2012Metric" H 5738 1250 50  0001 C CNN
 F 3 "~" H 5700 1400 50  0001 C CNN
@@
 Wire Wire Line
 	5700 1800 5700 1550
-Wire Wire Line
-	5700 1250 5700 1000
-Wire Wire Line
-	5700 1000 5600 1000
 $Comp
 L Device:C C1002
@@
 P 4000 1350
 F 0 "C1002" H 4115 1396 50  0000 L CNN
-F 1 "0.1uF" H 4115 1305 50  0000 L CNN
+F 1 "100nF" H 4115 1305 50  0000 L CNN
 F 2 "Capacitor_SMD:C_0805_2012Metric" H 4038 1200 50  0001 C CNN
 F 3 "~" H 4000 1350 50  0001 C CNN
@@
 P 6300 1400
 F 0 "C1007" H 6415 1446 50  0000 L CNN
-F 1 "33uF" H 6415 1355 50  0000 L CNN
+F 1 "47uF" H 6415 1355 50  0000 L CNN
 F 2 "Capacitor_SMD:C_0805_2012Metric" H 6338 1250 50  0001 C CNN
 F 3 "~" H 6300 1400 50  0001 C CNN
@@
 Wire Wire Line
 	5700 1800 5950 1800
-Wire Wire Line
-	5700 1000 6300 1000
-Connection ~ 5700 1000
 $Comp
 L power:GND #PWR01009
@@
 P 5800 2400
 F 0 "C1006" H 5915 2446 50  0000 L CNN
-F 1 "39pF" H 5915 2355 50  0000 L CNN
+F 1 "10pf" H 5915 2355 50  0000 L CNN
 F 2 "Capacitor_SMD:C_0805_2012Metric" H 5838 2250 50  0001 C CNN
 F 3 "~" H 5800 2400 50  0001 C CNN
@@
 P 5100 2150
 F 0 "C1004" H 5215 2196 50  0000 L CNN
-F 1 "4700pF" H 5215 2105 50  0000 L CNN
+F 1 "1nF" H 5215 2105 50  0000 L CNN
 F 2 "Capacitor_SMD:C_0805_2012Metric" H 5138 2000 50  0001 C CNN
 F 3 "~" H 5100 2150 50  0001 C CNN
@@
 P 5100 2450
 F 0 "R1003" H 5170 2496 50  0000 L CNN
-F 1 "44.9K" H 5170 2405 50  0000 L CNN
+F 1 "49.9k" H 5170 2405 50  0000 L CNN
 F 2 "Resistor_SMD:R_0805_2012Metric" V 5030 2450 50  0001 C CNN
 F 3 "~" H 5100 2450 50  0001 C CNN
@@
 P 6650 2100
 F 0 "R1004" H 6720 2146 50  0000 L CNN
-F 1 "10k" H 6720 2055 50  0000 L CNN
+F 1 "10.2k" H 6720 2055 50  0000 L CNN
 F 2 "Resistor_SMD:R_0805_2012Metric" V 6580 2100 50  0001 C CNN
 F 3 "~" H 6650 2100 50  0001 C CNN
@@
 	6650 2250 6650 2400
 Connection ~ 6650 2400
-Wire Wire Line
-	6650 1000 6300 1000
-Connection ~ 6300 1000
 $Comp
 L power:GND #PWR01010
@@
 	-1   0    0    1
 $EndComp
-Wire Wire Line
-	6900 1000 6650 1000
-Connection ~ 6650 1000
 $Comp
 L Device:C C1003
@@
 P 4000 2350
 F 0 "C1003" H 4115 2396 50  0000 L CNN
-F 1 "0.01uF" H 4115 2305 50  0000 L CNN
+F 1 "8.2nF" H 4115 2305 50  0000 L CNN
 F 2 "Capacitor_SMD:C_0805_2012Metric" H 4038 2200 50  0001 C CNN
 F 3 "~" H 4000 2350 50  0001 C CNN
@@
 P 2500 1950
 F 0 "C1001" H 2615 1996 50  0000 L CNN
-F 1 "4700pF" H 2615 1905 50  0000 L CNN
+F 1 "10uF" H 2615 1905 50  0000 L CNN
 F 2 "Capacitor_SMD:C_0805_2012Metric" H 2538 1800 50  0001 C CNN
 F 3 "~" H 2500 1950 50  0001 C CNN
 	1    2500 1950
-	1    0    0    -1
-$EndComp
-$Comp
-L Device:R R1001
-U 1 1 6140D70E
-P 3300 2050
-F 0 "R1001" H 3370 2096 50  0000 L CNN
-F 1 "332k" H 3370 2005 50  0000 L CNN
-F 2 "Resistor_SMD:R_0805_2012Metric" V 3230 2050 50  0001 C CNN
-F 3 "~" H 3300 2050 50  0001 C CNN
-	1    3300 2050
-	1    0    0    -1
-$EndComp
-$Comp
-L Device:R R1002
-U 1 1 6140DD86
-P 3300 2500
-F 0 "R1002" H 3370 2546 50  0000 L CNN
-F 1 "68.1k" H 3370 2455 50  0000 L CNN
-F 2 "Resistor_SMD:R_0805_2012Metric" V 3230 2500 50  0001 C CNN
-F 3 "~" H 3300 2500 50  0001 C CNN
-	1    3300 2500
 	1    0    0    -1
 $EndComp
@@
 $EndComp
 Wire Wire Line
-	3300 1900 3300 1800
-Connection ~ 3300 1800
-Wire Wire Line
-	3300 2200 3300 2250
-Wire Wire Line
-	3300 2650 3300 2700
-Wire Wire Line
-	3300 2700 4000 2700
-Wire Wire Line
 	4000 2500 4000 2700
-Connection ~ 4000 2700
-Wire Wire Line
-	3300 1800 4150 1800
 Wire Wire Line
 	4000 2200 4000 2000
 Wire Wire Line
 	4000 2000 4150 2000
-Wire Wire Line
-	4150 1900 3600 1900
-Wire Wire Line
-	3600 1900 3600 2250
-Wire Wire Line
-	3600 2250 3300 2250
-Connection ~ 3300 2250
-Wire Wire Line
-	3300 2250 3300 2350
 $Comp
 L power:GND #PWR01003
@@
 	0    1    1    0
 $EndComp
-$Comp
-L Connector:Conn_01x02_Male J1007
-U 1 1 61724ED0
-P 6850 1400
-F 0 "J1007" V 6912 1444 50  0000 L CNN
-F 1 "Conn_01x02_Male" V 7003 1444 50  0000 L CNN
-F 2 "Connector_PinHeader_2.54mm:PinHeader_1x02_P2.54mm_Vertical" H 6850 1400 50  0001 C CNN
-F 3 "~" H 6850 1400 50  0001 C CNN
-	1    6850 1400
-	-1   0    0    1
-$EndComp
-Wire Wire Line
-	6650 1000 6650 1300
-Wire Wire Line
-	6650 1400 6650 1950
-Wire Wire Line
-	1700 1800 2500 1800
+Wire Wire Line
+	1700 1800 2150 1800
 Connection ~ 2500 1800
-Wire Wire Line
-	2500 1800 3300 1800
-Text Notes 2550 3150 0    50   ~ 0
-R1001 and 1002 need to be changed to be a voltage divider\n
 $Comp
 L dk_Diodes-Rectifiers-Single:B340A-13-F D1002
@@
 $EndComp
 Wire Wire Line
-	4850 1000 5100 1000
-Wire Wire Line
 	4850 1800 5100 1800
 Wire Wire Line
 	5100 1150 5100 1000
-Connection ~ 5100 1000
-Wire Wire Line
-	5100 1000 5300 1000
 Wire Wire Line
 	5100 1550 5100 1800
@@
 Wire Wire Line
 	5100 1800 5700 1800
+$Comp
+L Device:C C1008
+U 1 1 61297C6F
+P 2150 1950
+F 0 "C1008" H 2265 1996 50  0000 L CNN
+F 1 "10uF" H 2265 1905 50  0000 L CNN
+F 2 "Capacitor_SMD:C_0805_2012Metric" H 2188 1800 50  0001 C CNN
+F 3 "~" H 2150 1950 50  0001 C CNN
+	1    2150 1950
+	1    0    0    -1
+$EndComp
+$Comp
+L power:GND #PWR0101
+U 1 1 61297C79
+P 2150 2100
+F 0 "#PWR0101" H 2150 1850 50  0001 C CNN
+F 1 "GND" H 2155 1927 50  0000 C CNN
+F 2 "" H 2150 2100 50  0001 C CNN
+F 3 "" H 2150 2100 50  0001 C CNN
+	1    2150 2100
+	1    0    0    -1
+$EndComp
+Connection ~ 2150 1800
+Wire Wire Line
+	2150 1800 2500 1800
+Wire Wire Line
+	2500 1800 4150 1800
+Wire Wire Line
+	4850 1000 5100 1000
+$Comp
+L SamacSys_Parts:SRN8040-100M L1001
+U 1 1 612C1A78
+P 5100 1000
+F 0 "L1001" H 5500 1225 50  0000 C CNN
+F 1 "SRN8040-100M" H 5500 1134 50  0000 C CNN
+F 2 "SamacSys_Parts:SRN8040100M" H 5750 1050 50  0001 L CNN
+F 3 "https://componentsearchengine.com/Datasheets/1/SRN8040-100M.pdf" H 5750 950 50  0001 L CNN
+F 4 "Bourns SRN8040 Series Type SMD Shielded Wire-wound SMD Inductor with a Ferrite Core, 10 uH +/-20% Semi-Shielded 3.1A Idc" H 5750 850 50  0001 L CNN "Description"
+F 5 "4" H 5750 750 50  0001 L CNN "Height"
+F 6 "652-SRN8040-100M" H 5750 650 50  0001 L CNN "Mouser Part Number"
+F 7 "https://www.mouser.co.uk/ProductDetail/Bourns/SRN8040-100M?qs=opBjA1TV901MvrktVUEKyA%3D%3D" H 5750 550 50  0001 L CNN "Mouser Price/Stock"
+F 8 "Bourns" H 5750 450 50  0001 L CNN "Manufacturer_Name"
+F 9 "SRN8040-100M" H 5750 350 50  0001 L CNN "Manufacturer_Part_Number"
+	1    5100 1000
+	1    0    0    -1
+$EndComp
+Connection ~ 5100 1000
+Wire Wire Line
+	5700 1250 5900 1250
+Wire Wire Line
+	5900 1250 5900 1000
+Wire Wire Line
+	5900 1000 6300 1000
+Connection ~ 5900 1000
+Connection ~ 6300 1000
+Wire Wire Line
+	6300 1000 6650 1000
+Wire Wire Line
+	6650 1600 6650 1950
+Wire Wire Line
+	6650 1300 6650 1000
+Connection ~ 6650 1000
+Wire Wire Line
+	6650 1000 6900 1000
+$Comp
+L Device:R R1001
+U 1 1 6134FCA9
+P 6650 1450
+F 0 "R1001" H 6720 1496 50  0000 L CNN
+F 1 "0" H 6720 1405 50  0000 L CNN
+F 2 "Resistor_SMD:R_0805_2012Metric" V 6580 1450 50  0001 C CNN
+F 3 "~" H 6650 1450 50  0001 C CNN
+	1    6650 1450
+	1    0    0    -1
+$EndComp
 $EndSCHEMATC

Commit message: V1.1 working progress
Implemented further documentation
New boost converter for the battery
power switches
Led indicator
removed unnecessary elements
Parts:
- removed D1001: 1N5400, Diode_THT:D_DO-201AD_P12.70mm_Horizontal, symbol Diode:1N5400
- removed J1001, J1002, J1008: Conn_01x02_Male, Connector_PinHeader_2.54mm:PinHeader_1x02_P2.54mm_Vertical, symbol Connector:Conn_01x02_Male
- removed J1005, J1006: Conn_01x06_Female, Connector_PinSocket_2.54mm:PinSocket_1x06_P2.54mm_Vertical, symbol Connector:Conn_01x06_Female
- removed J1013: Conn_02x04_Odd_Even, Connector_PinHeader_2.54mm:PinHeader_2x04_P2.54mm_Vertical, symbol Connector_Generic:Conn_02x04_Odd_Even
- removed L1001: SRN8040-100M, SamacSys_Parts:SRN8040100M, symbol SamacSys_Parts:SRN8040-100M
- removed Q1001: IRF9540N, digikey-footprints:TO-220-3, symbol Transistor_FET:IRF9540N
- added C10, C9: C, Capacitor_SMD:C_0805_2012Metric, symbol Device:C
- added C11: 22uf 3.71mohm, Capacitor_SMD:C_0805_2012Metric, symbol Device:C
- added C12: 10uf 3mohm, Capacitor_SMD:C_0805_2012Metric, symbol Device:C
- added D1: 1N5400, Diode_THT:D_DO-201AD_P12.70mm_Horizontal, symbol Diode:1N5400
- added D4: LTST-C190GKT, digikey-footprints:LED_0603, symbol dk_LED-Indication-Discrete:LTST-C190GKT
- added HW-1: Charger-New_Library-RackComm-rescue-RackComm-resc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, CI_ComPCB:Charger, symbol CI_ComPCB-rescue:Charger-New_Library-RackComm-rescue-RackComm-rescue
- added Holder1: Battery-New_Library-RackComm-rescue, CI_ComPCB:Battery, symbol CI_ComPCB-rescue:Battery-New_Library-RackComm-rescue
- added L1: SRN8040-100M, SamacSys_Parts:SRN8040100M, symbol SamacSys_Parts:SRN8040-100M
- added L2: SRN8040-R50Y, SamacSys_Parts:SRN8040R50Y, symbol SamacSys_Parts:SRN8040-R50Y
- added PS1: TPS63810YFFR, SamacSys_Parts:BGA15C40P3X5_134X226X62, symbol SamacSys_Parts:TPS63810YFFR
- added Q1: Transistor_FET_IRF9540N, Package_TO_SOT_THT:TO-220-3_Vertical, symbol CI_ComPCB-cache:Transistor_FET_IRF9540N
- added R9: 330, Resistor_SMD:R_0805_2012Metric, symbol Device:R
- added S1, S2: JS202011SCQN, digikey-footprints:Switch_Slide_JS202011SCQN, symbol dk_Slide-Switches:JS202011SCQN
- added SW1: SW_SPDT, digikey-footprints:Switch_Toggle_ATE1D-2M3-10-Z, symbol Switch:SW_SPDT
- added SW2: SW_DIP_x04, Button_Switch_SMD:SW_DIP_SPSTx04_Slide_9.78x12.34mm_W8.61mm_P2.54mm, symbol Switch:SW_DIP_x04
- R2: renamed from R1006; value 330 -> 680
- R3: renamed from R1007; value 330 -> 680
- R4: renamed from R1008; value 330 -> 680
- R5: renamed from R1009; value 330 -> 680
- renumbered C1008 to C1, C1001 to C2, C1002 to C3, C1003 to C4, C1004 to C5, C1005 to C6, C1006 to C7, C1007 to C8, Converter1001 to Converter1, Converter1002 to Converter2, D1002 to D2, D1003 to D3, J1003 to J3, J1004 to J4, J1009 to J5, J1010 to J6, J1011 to J7, J1012 to J8, R1003 to R1, R1001 to R6, R1004 to R7, R1005 to R8, U1001 to U1, U1002 to U2
Connections:
- net labels added: B_SW1, Battery_Power, Buck_Out, Charger_GND, Charger_IN, Charger_OUT, ESP_Power
- wire segments 169 -> 179
- no-connect marks 6 -> 2
Other:
- note added: "12v to 5v converter"
- note added: "4.2 to 5v converter"
- note added: "Charger"
- note added: "Device ON/OFF Switch"
- note added: "Power To/From Rack switch"
- note added: "change switch to \nCS12ANW03"
- note added: "change switches to \nCS22BNW03"
- moved on the sheet: C1, C2, C3, C4, C5, C6, C7, C8, Converter1, Converter2, D2, J3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

Commit message: V1.1 in development
Implemented sheets
Added correct switches
Completed boost converter
REQUIRED before build:
PCB layout
Component matching with PCB maker
Parts:
- removed C1, C2: 10uF, Capacitor_SMD:C_0805_2012Metric, symbol Device:C
- removed C10, C9: C, Capacitor_SMD:C_0805_2012Metric, symbol Device:C
- removed C11: 22uf 3.71mohm, Capacitor_SMD:C_0805_2012Metric, symbol Device:C
- removed C12: 10uf 3mohm, Capacitor_SMD:C_0805_2012Metric, symbol Device:C
- removed C3: 100nF, Capacitor_SMD:C_0805_2012Metric, symbol Device:C
- removed C4: 8.2nF, Capacitor_SMD:C_0805_2012Metric, symbol Device:C
- removed C5: 1nF, Capacitor_SMD:C_0805_2012Metric, symbol Device:C
- removed C6, C8: 47uF, Capacitor_SMD:C_0805_2012Metric, symbol Device:C
- removed C7: 10pf, Capacitor_SMD:C_0805_2012Metric, symbol Device:C
- removed Converter1, Converter2: TxRx-RS485, CI_ComPCB:TXRX-AB, symbol CI_ComPCB-rescue:TxRx-RS485-New_Library-RackComm-rescue
- removed D1, D3: 1N5400, Diode_THT:D_DO-201AD_P12.70mm_Horizontal, symbol Diode:1N5400
- removed D2: B340A-13-F, digikey-footprints:DO-214AC, symbol dk_Diodes-Rectifiers-Single:B340A-13-F
- removed D4: LTST-C190GKT, digikey-footprints:LED_0603, symbol dk_LED-Indication-Discrete:LTST-C190GKT
- removed HW-1: Charger-New_Library-RackComm-rescue-RackComm-resc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, CI_ComPCB:Charger, symbol CI_ComPCB-rescue:Charger-New_Library-RackComm-rescue-RackComm-rescue
- removed Holder1: Battery-New_Library-RackComm-rescue, CI_ComPCB:Battery, symbol CI_ComPCB-rescue:Battery-New_Library-RackComm-rescue
- removed J5, J6: RJ45_LED_Shielded, Connector_RJ:RJ45_Amphenol_RJHSE538X, symbol Connector:RJ45_LED_Shielded
- removed J7, J8: Conn_01x01_Female, Connector_PinHeader_2.54mm:PinHeader_1x01_P2.54mm_Vertical, symbol Connector:Conn_01x01_Female
- removed L1: SRN8040-100M, SamacSys_Parts:SRN8040100M, symbol SamacSys_Parts:SRN8040-100M
- removed L2: SRN8040-R50Y, SamacSys_Parts:SRN8040R50Y, symbol SamacSys_Parts:SRN8040-R50Y
- removed PS1: TPS63810YFFR, SamacSys_Parts:BGA15C40P3X5_134X226X62, symbol SamacSys_Parts:TPS63810YFFR
- removed Q1: Transistor_FET_IRF9540N, Package_TO_SOT_THT:TO-220-3_Vertical, symbol CI_ComPCB-cache:Transistor_FET_IRF9540N
- removed R1: 49.9k, Resistor_SMD:R_0805_2012Metric, symbol Device:R
- removed R2, R3, R4, R5: 680, Resistor_SMD:R_0805_2012Metric, symbol Device:R
- removed R6: 0, Resistor_SMD:R_0805_2012Metric, symbol Device:R
- removed R7: 10.2k, Resistor_SMD:R_0805_2012Metric, symbol Device:R
- removed R8: 1.91k, Resistor_SMD:R_0805_2012Metric, symbol Device:R
- removed R9: 330, Resistor_SMD:R_0805_2012Metric, symbol Device:R
- removed S1, S2: JS202011SCQN, digikey-footprints:Switch_Slide_JS202011SCQN, symbol dk_Slide-Switches:JS202011SCQN
- removed SW1: SW_SPDT, digikey-footprints:Switch_Toggle_ATE1D-2M3-10-Z, symbol Switch:SW_SPDT
- removed SW2: SW_DIP_x04, Button_Switch_SMD:SW_DIP_SPSTx04_Slide_9.78x12.34mm_W8.61mm_P2.54mm, symbol Switch:SW_DIP_x04
- removed U2: TPS54331, Package_SO:TI_SO-PowerPAD-8, symbol CI_ComPCB-rescue:TPS54331
- added D101: LTST-C190GKT, digikey-footprints:LED_0603, symbol dk_LED-Indication-Discrete:LTST-C190GKT
- added D102: B340A-13-F, digikey-footprints:DO-214AC, symbol dk_Diodes-Rectifiers-Single:B340A-13-F
- added R101: 680, Resistor_SMD:R_0805_2012Metric, symbol Device:R
- added S101, S102: CS22BNW03, SamacSys_Parts:CS22BNW03, symbol SamacSys_Parts:CS22BNW03
- added S103: CS12ANW03, SamacSys_Parts:CS12ANW03, symbol SamacSys_Parts:CS12ANW03
- renumbered J3 to J101, J4 to J102, U1 to U101
Connections:
- net labels added: Buck_Converter_OUT, Buck_IN
- net labels removed: A0, A1, B0, B1, Charger_GND, Charger_OUT, Sheild
- wire segments 179 -> 41
- no-connect marks 2 -> 3
Other:
- note added: "CI Communication PCB"
- note added: "Charging/Delivering Battery Power Switch"
- note removed: "12v to 5v converter"
- note removed: "4.2 to 5v converter"
- note removed: "Charger"
- note removed: "change switch to \nCS12ANW03"
- note removed: "change switches to \nCS22BNW03"
- moved on the sheet: J101, J102, U101
