File: CI_ComPCB/CI_ComPCB.sch (KiCad schematic (older format))
At the start: 6 parts, among them J101 Conn_01x01_Male, U101 ESP32s

Commit message: prilim pcb finished
Parts:
- added U102: oled(128x64)i2c, CI_ComPCB:oled(128x64)i2c, symbol oleds:oled(128x64)i2c
Connections:
- net 3.3V: now also U102.2 (VCC)
- net GND: now also U102.1 (GND)
- net at U101.D21: now also U102.4 (SDA)
- net at U101.D22: now also U102.3 (SCL)
Changed lines of the file:
@@
 Wire Wire Line
 	4411 4320 4850 4320
+$Comp
+L oleds:oled(128x64)i2c U102
+U 1 1 626EBE2D
+P 7650 4050
+F 0 "U102" H 8128 4054 50  0000 L CNN
+F 1 "oled(128x64)i2c" H 8128 3963 50  0000 L CNN
+F 2 "CI_ComPCB:oled(128x64)i2c" H 7650 3850 50  0001 C CNN
+F 3 "" H 7650 3850 50  0001 C CNN
+	1    7650 4050
+	-1   0    0    -1
+$EndComp
+Text GLabel 7900 3800 1    50   Input ~ 0
+GND
+Text GLabel 7750 3800 1    50   Input ~ 0
+3.3V
+Wire Wire Line
+	6350 3020 7600 3020
+Wire Wire Line
+	7600 3020 7600 3800
+Wire Wire Line
+	7450 3800 7450 3320
+Wire Wire Line
+	7450 3320 6350 3320
 $EndSCHEMATC
