File: CI_ComPCB/12v to 5v Converter.sch (KiCad schematic (older format))
At the start: 18 parts, among them IC401 TPS54331DR, J401 Connector_Conn_01x01_Male, J402 Conn_01x02_Male, J403 Conn_01x01_Male

Commit message: Sensor_SplitterPrint
Parts:
- D401, D402: symbol CI_ComPCB-rescue:SS34-SamacSys_Parts -> CI_ComPCB-rescue:SS34-SamacSys_Parts-CI_ComPCB-rescue
- IC401: symbol CI_ComPCB-rescue:TPS54331DR-SamacSys_Parts -> CI_ComPCB-rescue:TPS54331DR-SamacSys_Parts-CI_ComPCB-rescue
- J401: symbol CI_ComPCB-cache:Connector_Conn_01x01_Male -> CI_ComPCB-rescue:Connector_Conn_01x01_Male-CI_ComPCB-cache
- L401: symbol CI_ComPCB-rescue:RLF12560T-7R8N8R2-SamacSys_Parts -> CI_ComPCB-rescue:RLF12560T-7R8N8R2-SamacSys_Parts-CI_ComPCB-rescue
Changed lines of the file:
@@
 Buck_IN
 $Comp
-L CI_ComPCB-rescue:SS34-SamacSys_Parts D402
+L CI_ComPCB-rescue:SS34-SamacSys_Parts-CI_ComPCB-rescue D402
 U 1 1 612967EC
 P 8100 2850
@@
 	5600 3650 5850 3650
 $Comp
-L CI_ComPCB-rescue:SS34-SamacSys_Parts D401
+L CI_ComPCB-rescue:SS34-SamacSys_Parts-CI_ComPCB-rescue D401
 U 1 1 6129D4B6
 P 5850 2900
@@
 	7400 2850 7400 3440
 $Comp
-L CI_ComPCB-rescue:RLF12560T-7R8N8R2-SamacSys_Parts L401
+L CI_ComPCB-rescue:RLF12560T-7R8N8R2-SamacSys_Parts-CI_ComPCB-rescue L401
 U 1 1 612ACFD5
 P 5850 2850
@@
 Connection ~ 6650 2850
 $Comp
-L CI_ComPCB-rescue:TPS54331DR-SamacSys_Parts IC401
+L CI_ComPCB-rescue:TPS54331DR-SamacSys_Parts-CI_ComPCB-rescue IC401
 U 1 1 612C5C0D
 P 4400 3550
@@
 $EndComp
 $Comp
-L CI_ComPCB-cache:Connector_Conn_01x01_Male J401
+L CI_ComPCB-rescue:Connector_Conn_01x01_Male-CI_ComPCB-cache J401
 U 1 1 614D9F4C
 P 3210 3450
+AR Path="/614D9F4C" Ref="J401"  Part="1"
+AR Path="/61A31DC2/614D9F4C" Ref="J401"  Part="1"
 F 0 "J401" V 3272 3494 50  0000 L CNN
 F 1 "Connector_Conn_01x01_Male" V 3363 3494 50  0000 L CNN
