File: CI_ComPCB/12v to 5v Converter.sch (KiCad schematic (older format))
At the start: 18 parts, among them IC401 TPS54331DR, J401 Connector_Conn_01x01_Male, J402 Conn_01x02_Male, J403 Conn_01x01_Male

Commit message: Production1
Parts:
- removed J402: Conn_01x02_Male, Connector_PinHeader_2.54mm:PinHeader_1x02_P2.54mm_Vertical, symbol Connector:Conn_01x02_Male
- D201: renamed from D401; symbol CI_ComPCB-rescue:SS34-SamacSys_Parts -> CI_ComPCB-rescue:SS34-SamacSys_Parts-CI_ComPCB-rescue
- D202: renamed from D402; symbol CI_ComPCB-rescue:SS34-SamacSys_Parts -> CI_ComPCB-rescue:SS34-SamacSys_Parts-CI_ComPCB-rescue
- IC201: renamed from IC401; symbol CI_ComPCB-rescue:TPS54331DR-SamacSys_Parts -> CI_ComPCB-rescue:TPS54331DR-SamacSys_Parts-CI_ComPCB-rescue
- J201: renamed from J401; symbol CI_ComPCB-cache:Connector_Conn_01x01_Male -> CI_ComPCB-rescue:Connector_Conn_01x01_Male-CI_ComPCB-cache
- L201: renamed from L401; symbol CI_ComPCB-rescue:RLF12560T-7R8N8R2-SamacSys_Parts -> CI_ComPCB-rescue:RLF12560T-7R8N8R2-SamacSys_Parts-CI_ComPCB-rescue
- renumbered C401 to C201, C402 to C202, C403 to C203, C404 to C204, C405 to C205, C406 to C206, C407 to C207, C408 to C208, J403 to J202, R401 to R201, R403 to R202, R404 to R203
Connections:
- net labels added: EPower
- net labels removed: Buck_IN
Changed lines of the file:
@@
 $Descr A4 11693 8268
 encoding utf-8
-Sheet 4 6
+Sheet 2 3
 Title ""
 Date ""
@@
 P 6450 3250
 AR Path="/61A8D138" Ref="C?"  Part="1"
-AR Path="/61A31DC2/61A8D138" Ref="C406"  Part="1"
-F 0 "C406" H 6565 3296 50  0000 L CNN
+AR Path="/61A31DC2/61A8D138" Ref="C206"  Part="1"
+F 0 "C206" H 6565 3296 50  0000 L CNN
 F 1 "47uF" H 6565 3205 50  0000 L CNN
 F 2 "Capacitor_SMD:C_0805_2012Metric" H 6488 3100 50  0001 C CNN
@@
 P 4250 3200
 AR Path="/61A8D13F" Ref="C?"  Part="1"
-AR Path="/61A31DC2/61A8D13F" Ref="C403"  Part="1"
-F 0 "C403" H 4365 3246 50  0000 L CNN
+AR Path="/61A31DC2/61A8D13F" Ref="C203"  Part="1"
+F 0 "C203" H 4365 3246 50  0000 L CNN
 F 1 "100nF" H 4365 3155 50  0000 L CNN
 F 2 "Capacitor_SMD:C_0805_2012Metric" H 4288 3050 50  0001 C CNN
@@
 P 7050 3250
 AR Path="/61A8D146" Ref="C?"  Part="1"
-AR Path="/61A31DC2/61A8D146" Ref="C408"  Part="1"
-F 0 "C408" H 7165 3296 50  0000 L CNN
+AR Path="/61A31DC2/61A8D146" Ref="C208"  Part="1"
+F 0 "C208" H 7165 3296 50  0000 L CNN
 F 1 "47uF" H 7165 3205 50  0000 L CNN
 F 2 "Capacitor_SMD:C_0805_2012Metric" H 7088 3100 50  0001 C CNN
@@
 P 6550 4250
 AR Path="/61A8D158" Ref="C?"  Part="1"
-AR Path="/61A31DC2/61A8D158" Ref="C407"  Part="1"
-F 0 "C407" H 6665 4296 50  0000 L CNN
+AR Path="/61A31DC2/61A8D158" Ref="C207"  Part="1"
+F 0 "C207" H 6665 4296 50  0000 L CNN
 F 1 "10pf" H 6665 4205 50  0000 L CNN
 F 2 "Capacitor_SMD:C_0805_2012Metric" H 6588 4100 50  0001 C CNN
@@
 P 5850 4000
 AR Path="/61A8D160" Ref="C?"  Part="1"
-AR Path="/61A31DC2/61A8D160" Ref="C405"  Part="1"
-F 0 "C405" H 5965 4046 50  0000 L CNN
+AR Path="/61A31DC2/61A8D160" Ref="C205"  Part="1"
+F 0 "C205" H 5965 4046 50  0000 L CNN
 F 1 "1nF" H 5965 3955 50  0000 L CNN
 F 2 "Capacitor_SMD:C_0805_2012Metric" H 5888 3850 50  0001 C CNN
@@
 P 5850 4300
 AR Path="/61A8D169" Ref="R?"  Part="1"
-AR Path="/61A31DC2/61A8D169" Ref="R401"  Part="1"
-F 0 "R401" H 5920 4346 50  0000 L CNN
+AR Path="/61A31DC2/61A8D169" Ref="R201"  Part="1"
+F 0 "R201" H 5920 4346 50  0000 L CNN
 F 1 "56.2k" H 5920 4255 50  0000 L CNN
 F 2 "Resistor_SMD:R_0805_2012Metric" V 5780 4300 50  0001 C CNN
@@
 P 7400 3590
 AR Path="/61A8D17A" Ref="R?"  Part="1"
-AR Path="/61A31DC2/61A8D17A" Ref="R403"  Part="1"
-F 0 "R403" H 7470 3636 50  0000 L CNN
+AR Path="/61A31DC2/61A8D17A" Ref="R202"  Part="1"
+F 0 "R202" H 7470 3636 50  0000 L CNN
 F 1 "10.2k" H 7470 3545 50  0000 L CNN
 F 2 "Resistor_SMD:R_0805_2012Metric" V 7330 3590 50  0001 C CNN
@@
 P 4250 4200
 AR Path="/61A8D195" Ref="C?"  Part="1"
-AR Path="/61A31DC2/61A8D195" Ref="C404"  Part="1"
-F 0 "C404" H 4365 4246 50  0000 L CNN
+AR Path="/61A31DC2/61A8D195" Ref="C204"  Part="1"
+F 0 "C204" H 4365 4246 50  0000 L CNN
 F 1 "8.2nF" H 4365 4155 50  0000 L CNN
 F 2 "Capacitor_SMD:C_0603_1608Metric" H 4288 4050 50  0001 C CNN
@@
 P 3900 3800
 AR Path="/61A8D19B" Ref="C?"  Part="1"
-AR Path="/61A31DC2/61A8D19B" Ref="C402"  Part="1"
-F 0 "C402" H 4015 3846 50  0000 L CNN
+AR Path="/61A31DC2/61A8D19B" Ref="C202"  Part="1"
+F 0 "C202" H 4015 3846 50  0000 L CNN
 F 1 "10uF" H 4015 3755 50  0000 L CNN
 F 2 "Capacitor_SMD:C_0805_2012Metric" H 3938 3650 50  0001 C CNN
@@
 P 3520 3800
 AR Path="/61A8D1B6" Ref="C?"  Part="1"
-AR Path="/61A31DC2/61A8D1B6" Ref="C401"  Part="1"
-F 0 "C401" H 3635 3846 50  0000 L CNN
+AR Path="/61A31DC2/61A8D1B6" Ref="C201"  Part="1"
+F 0 "C201" H 3635 3846 50  0000 L CNN
 F 1 "10uF" H 3635 3755 50  0000 L CNN
 F 2 "Capacitor_SMD:C_0805_2012Metric" H 3558 3650 50  0001 C CNN
@@
 Text Notes 7370 7500 0    50   ~ 0
 12v to 5v converter
-Text GLabel 8100 2850 2    50   Input ~ 0
+Text GLabel 8000 2850 2    50   Input ~ 0
 Vin
 Text Notes 7060 7090 0    50   ~ 0
@@
 	3520 3650 3900 3650
 Text GLabel 3210 3650 0    50   Input ~ 0
-Buck_IN
-$Comp
-L CI_ComPCB-rescue:SS34-SamacSys_Parts D402
+EPower
+$Comp
+L CI_ComPCB-rescue:SS34-SamacSys_Parts-CI_ComPCB-rescue D202
 U 1 1 612967EC
 P 8100 2850
-F 0 "D402" H 8500 2583 50  0000 C CNN
+F 0 "D202" H 8500 2583 50  0000 C CNN
 F 1 "SS34" H 8500 2674 50  0000 C CNN
 F 2 "digikey-footprints:DO-214AC" H 8600 3000 50  0001 L CNN
@@
 	5600 3650 5850 3650
 $Comp
-L CI_ComPCB-rescue:SS34-SamacSys_Parts D401
+L CI_ComPCB-rescue:SS34-SamacSys_Parts-CI_ComPCB-rescue D201
 U 1 1 6129D4B6
 P 5850 2900
-F 0 "D401" H 6250 2633 50  0000 C CNN
+F 0 "D201" H 6250 2633 50  0000 C CNN
 F 1 "SS34" H 6250 2724 50  0000 C CNN
 F 2 "digikey-footprints:DO-214AC" H 6350 3050 50  0001 L CNN
@@
 	7400 2850 7400 3440
 $Comp
-L CI_ComPCB-rescue:RLF12560T-7R8N8R2-SamacSys_Parts L401
+L CI_ComPCB-rescue:RLF12560T-7R8N8R2-SamacSys_Parts-CI_ComPCB-rescue L201
 U 1 1 612ACFD5
 P 5850 2850
-F 0 "L401" H 6250 3075 50  0000 C CNN
+F 0 "L201" H 6250 3075 50  0000 C CNN
 F 1 "RLF12560T-7R8N8R2" H 6250 2984 50  0000 C CNN
 F 2 "SamacSys_Parts:INDPM128125X600N" H 6500 2900 50  0001 L CNN
@@
 Connection ~ 6650 2850
 $Comp
-L CI_ComPCB-rescue:TPS54331DR-SamacSys_Parts IC401
+L CI_ComPCB-rescue:TPS54331DR-SamacSys_Parts-CI_ComPCB-rescue IC201
 U 1 1 612C5C0D
 P 4400 3550
-F 0 "IC401" H 5000 3815 50  0000 C CNN
+F 0 "IC201" H 5000 3815 50  0000 C CNN
 F 1 "TPS54331DR" H 5000 3724 50  0000 C CNN
 F 2 "SamacSys_Parts:SOIC127P600X175-8N" H 5450 3650 50  0001 L CNN
@@
 P 6700 3650
 AR Path="/61A8D150" Ref="#PWR?"  Part="1"
-AR Path="/61A31DC2/61A8D150" Ref="#PWR0405"  Part="1"
-F 0 "#PWR0405" H 6700 3400 50  0001 C CNN
+AR Path="/61A31DC2/61A8D150" Ref="#PWR0205"  Part="1"
+F 0 "#PWR0205" H 6700 3400 50  0001 C CNN
 F 1 "GND" H 6705 3477 50  0000 C CNN
 F 2 "" H 6700 3650 50  0001 C CNN
@@
 P 6200 4700
 AR Path="/61A8D172" Ref="#PWR?"  Part="1"
-AR Path="/61A31DC2/61A8D172" Ref="#PWR0404"  Part="1"
-F 0 "#PWR0404" H 6200 4450 50  0001 C CNN
+AR Path="/61A31DC2/61A8D172" Ref="#PWR0204"  Part="1"
+F 0 "#PWR0204" H 6200 4450 50  0001 C CNN
 F 1 "GND" H 6205 4527 50  0000 C CNN
 F 2 "" H 6200 4700 50  0001 C CNN
@@
 P 7400 4900
 AR Path="/61A8D18E" Ref="#PWR?"  Part="1"
-AR Path="/61A31DC2/61A8D18E" Ref="#PWR0406"  Part="1"
-F 0 "#PWR0406" H 7400 4650 50  0001 C CNN
+AR Path="/61A31DC2/61A8D18E" Ref="#PWR0206"  Part="1"
+F 0 "#PWR0206" H 7400 4650 50  0001 C CNN
 F 1 "GND" H 7405 4727 50  0000 C CNN
 F 2 "" H 7400 4900 50  0001 C CNN
@@
 P 7400 4550
 AR Path="/61A8D180" Ref="R?"  Part="1"
-AR Path="/61A31DC2/61A8D180" Ref="R404"  Part="1"
-F 0 "R404" H 7470 4596 50  0000 L CNN
+AR Path="/61A31DC2/61A8D180" Ref="R203"  Part="1"
+F 0 "R203" H 7470 4596 50  0000 L CNN
 F 1 "1.78k" H 7470 4505 50  0000 L CNN
 F 2 "Resistor_SMD:R_0805_2012Metric" V 7330 4550 50  0001 C CNN
@@
 P 4250 4550
 AR Path="/61A8D1A1" Ref="#PWR?"  Part="1"
-AR Path="/61A31DC2/61A8D1A1" Ref="#PWR0403"  Part="1"
-F 0 "#PWR0403" H 4250 4300 50  0001 C CNN
+AR Path="/61A31DC2/61A8D1A1" Ref="#PWR0203"  Part="1"
+F 0 "#PWR0203" H 4250 4300 50  0001 C CNN
 F 1 "GND" H 4255 4377 50  0000 C CNN
 F 2 "" H 4250 4550 50  0001 C CNN
@@
 P 3900 3950
 AR Path="/61A8D1AA" Ref="#PWR?"  Part="1"
-AR Path="/61A31DC2/61A8D1AA" Ref="#PWR0402"  Part="1"
-F 0 "#PWR0402" H 3900 3700 50  0001 C CNN
+AR Path="/61A31DC2/61A8D1AA" Ref="#PWR0202"  Part="1"
+F 0 "#PWR0202" H 3900 3700 50  0001 C CNN
 F 1 "GND" H 3905 3777 50  0000 C CNN
 F 2 "" H 3900 3950 50  0001 C CNN
@@
 P 3520 3950
 AR Path="/61A8D1BC" Ref="#PWR?"  Part="1"
-AR Path="/61A31DC2/61A8D1BC" Ref="#PWR0401"  Part="1"
-F 0 "#PWR0401" H 3520 3700 50  0001 C CNN
+AR Path="/61A31DC2/61A8D1BC" Ref="#PWR0201"  Part="1"
+F 0 "#PWR0201" H 3520 3700 50  0001 C CNN
 F 1 "GND" H 3525 3777 50  0000 C CNN
 F 2 "" H 3520 3950 50  0001 C CNN
@@
 $EndComp
 $Comp
-L CI_ComPCB-cache:Connector_Conn_01x01_Male J401
+L CI_ComPCB-rescue:Connector_Conn_01x01_Male-CI_ComPCB-cache J?
 U 1 1 614D9F4C
 P 3210 3450
-F 0 "J401" V 3272 3494 50  0000 L CNN
+AR Path="/614D9F4C" Ref="J?"  Part="1"
+AR Path="/61A31DC2/614D9F4C" Ref="J201"  Part="1"
+F 0 "J201" V 3272 3494 50  0000 L CNN
 F 1 "Connector_Conn_01x01_Male" V 3363 3494 50  0000 L CNN
 F 2 "Connector_PinHeader_2.54mm:PinHeader_1x01_P2.54mm_Vertical" H 3210 3450 50  0001 C CNN
@@
 $EndComp
 $Comp
-L Connector:Conn_01x02_Male J402
-U 1 1 61839510
-P 8100 2650
-F 0 "J402" V 8162 2694 50  0000 L CNN
-F 1 "Conn_01x02_Male" V 8253 2694 50  0000 L CNN
-F 2 "Connector_PinHeader_2.54mm:PinHeader_1x02_P2.54mm_Vertical" H 8100 2650 50  0001 C CNN
-F 3 "~" H 8100 2650 50  0001 C CNN
-	1    8100 2650
-	0    1    1    0
-$EndComp
-$Comp
-L Connector:Conn_01x01_Male J403
+L Connector:Conn_01x01_Male J202
 U 1 1 6184D048
 P 4776 4344
-F 0 "J403" H 4884 4525 50  0000 C CNN
+F 0 "J202" H 4884 4525 50  0000 C CNN
 F 1 "Conn_01x01_Male" H 4884 4434 50  0000 C CNN
 F 2 "Connector_PinHeader_2.54mm:PinHeader_1x01_P2.54mm_Vertical" H 4776 4344 50  0001 C CNN

Commit message: print
Parts:
- removed L201: RLF12560T-7R8N8R2, SamacSys_Parts:INDPM128125X600N, symbol CI_ComPCB-rescue:RLF12560T-7R8N8R2-SamacSys_Parts-CI_ComPCB-rescue
- added L201: IHLP2525CZER6R8M01, IND:IHLP2525CZER6R8M01, symbol IHLP2525CZER6R8M01:IHLP2525CZER6R8M01
- C201, C202: value 10uF -> 22uf; footprint Capacitor_SMD:C_0805_2012Metric -> Capacitor_SMD:C_1210_3225Metric
- C206, C208: footprint Capacitor_SMD:C_0805_2012Metric -> Capacitor_SMD:C_1210_3225Metric
Connections:
- net at C206.1, C208.1, D202.2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: now also L201.1
- net at C203.1, D201.1, IC201.8 (PH): now also L201.2
Changed lines of the file:
@@
 F 0 "C206" H 6565 3296 50  0000 L CNN
 F 1 "47uF" H 6565 3205 50  0000 L CNN
-F 2 "Capacitor_SMD:C_0805_2012Metric" H 6488 3100 50  0001 C CNN
+F 2 "Capacitor_SMD:C_1210_3225Metric" H 6488 3100 50  0001 C CNN
 F 3 "~" H 6450 3250 50  0001 C CNN
 	1    6450 3250
@@
 F 0 "C208" H 7165 3296 50  0000 L CNN
 F 1 "47uF" H 7165 3205 50  0000 L CNN
-F 2 "Capacitor_SMD:C_0805_2012Metric" H 7088 3100 50  0001 C CNN
+F 2 "Capacitor_SMD:C_1210_3225Metric" H 7088 3100 50  0001 C CNN
 F 3 "~" H 7050 3250 50  0001 C CNN
 	1    7050 3250
@@
 AR Path="/61A31DC2/61A8D19B" Ref="C202"  Part="1"
 F 0 "C202" H 4015 3846 50  0000 L CNN
-F 1 "10uF" H 4015 3755 50  0000 L CNN
-F 2 "Capacitor_SMD:C_0805_2012Metric" H 3938 3650 50  0001 C CNN
+F 1 "22uf" H 4015 3755 50  0000 L CNN
+F 2 "Capacitor_SMD:C_1210_3225Metric" H 3938 3650 50  0001 C CNN
 F 3 "~" H 3900 3800 50  0001 C CNN
 	1    3900 3800
@@
 AR Path="/61A31DC2/61A8D1B6" Ref="C201"  Part="1"
 F 0 "C201" H 3635 3846 50  0000 L CNN
-F 1 "10uF" H 3635 3755 50  0000 L CNN
-F 2 "Capacitor_SMD:C_0805_2012Metric" H 3558 3650 50  0001 C CNN
+F 1 "22uf" H 3635 3755 50  0000 L CNN
+F 2 "Capacitor_SMD:C_1210_3225Metric" H 3558 3650 50  0001 C CNN
 F 3 "~" H 3520 3800 50  0001 C CNN
 	1    3520 3800
@@
 $EndComp
 Wire Wire Line
-	5600 2850 5850 2850
+	5600 2850 5849 2850
 Wire Wire Line
 	6450 3100 6650 3100
@@
 	6650 3100 6650 2850
 Wire Wire Line
-	6650 2850 7050 2850
+	6650 2850 6652 2850
 Connection ~ 7050 2850
 Wire Wire Line
@@
 	7400 2850 7400 3440
 $Comp
-L CI_ComPCB-rescue:RLF12560T-7R8N8R2-SamacSys_Parts-CI_ComPCB-rescue L201
-U 1 1 612ACFD5
-P 5850 2850
-F 0 "L201" H 6250 3075 50  0000 C CNN
-F 1 "RLF12560T-7R8N8R2" H 6250 2984 50  0000 C CNN
-F 2 "SamacSys_Parts:INDPM128125X600N" H 6500 2900 50  0001 L CNN
-F 3 "https://product.tdk.com/system/files/dam/doc/product/inductor/inductor/smd/catalog/inductor_commercial_power_rlf12560_en.pdf" H 6500 2800 50  0001 L CNN
-F 4 "TDK - RLF12560T-7R8N8R2 - Power Inductor (SMD), 7.8 H, 8.4 A, Wirewound, 8.2 A, 12.8mm x 12.5mm x 6mm" H 6500 2700 50  0001 L CNN "Description"
-F 5 "6" H 6500 2600 50  0001 L CNN "Height"
-F 6 "810-RLF12560T-7R8N" H 6500 2500 50  0001 L CNN "Mouser Part Number"
-F 7 "https://www.mouser.co.uk/ProductDetail/TDK/RLF12560T-7R8N8R2?qs=3POhL7GGTOgHxYsYtKxdfg%3D%3D" H 6500 2400 50  0001 L CNN "Mouser Price/Stock"
-F 8 "TDK" H 6500 2300 50  0001 L CNN "Manufacturer_Name"
-F 9 "RLF12560T-7R8N8R2" H 6500 2200 50  0001 L CNN "Manufacturer_Part_Number"
-	1    5850 2850
-	1    0    0    -1
-$EndComp
-Connection ~ 5850 2850
-Connection ~ 6650 2850
-$Comp
 L CI_ComPCB-rescue:TPS54331DR-SamacSys_Parts-CI_ComPCB-rescue IC201
 U 1 1 612C5C0D
@@
 Wire Wire Line
 	4250 4544 4250 4550
+$Comp
+L IHLP2525CZER6R8M01:IHLP2525CZER6R8M01 L201
+U 1 1 61E06FC7
+P 5962 2849
+F 0 "L201" H 6262 3138 60  0000 C CNN
+F 1 "IHLP2525CZER6R8M01" H 6262 3032 60  0000 C CNN
+F 2 "IND:IHLP2525CZER6R8M01" H 6237 2564 60  0001 C CNN
+F 3 "" H 5962 2849 60  0000 C CNN
+	1    5962 2849
+	1    0    0    -1
+$EndComp
+Wire Wire Line
+	5962 2849 5849 2849
+Wire Wire Line
+	5849 2849 5849 2850
+Connection ~ 5849 2850
+Wire Wire Line
+	5849 2850 5850 2850
+Wire Wire Line
+	6562 2849 6652 2849
+Wire Wire Line
+	6652 2849 6652 2850
+Connection ~ 6652 2850
+Wire Wire Line
+	6652 2850 7050 2850
 $EndSCHEMATC

Commit message: prilim pcb finished
Parts:
- added F201: MF-MSMF050-2, SamacSys_Parts:FUSC4632X85N, symbol SamacSys_Parts:MF-MSMF050-2
- added RT201: SL08_10001, SamacSys_Parts:SL0810001, symbol SamacSys_Parts:SL08_10001
- L201: symbol IHLP2525CZER6R8M01:IHLP2525CZER6R8M01 -> CI_ComPCB-rescue:IHLP2525CZER6R8M01-IHLP2525CZER6R8M01
Connections:
- net EPower: now also F201.1; no longer C201.1, C202.1, IC201.2 (VIN), J201.1 (Pin_1)
- new net: C201.1, C202.1, IC201.2 (VIN), J201.1 (Pin_1), RT201.2
- new net: F201.2, RT201.1
Other:
- note added: "Current limiting circuit"
Changed lines of the file:
@@
 Wire Wire Line
 	3520 3650 3900 3650
-Text GLabel 3210 3650 0    50   Input ~ 0
+Text GLabel 1340 3650 0    50   Input ~ 0
 EPower
 $Comp
@@
 	4250 4544 4250 4550
 $Comp
-L IHLP2525CZER6R8M01:IHLP2525CZER6R8M01 L201
+L CI_ComPCB-rescue:IHLP2525CZER6R8M01-IHLP2525CZER6R8M01 L201
 U 1 1 61E06FC7
 P 5962 2849
+AR Path="/61E06FC7" Ref="L201"  Part="1"
+AR Path="/61A31DC2/61E06FC7" Ref="L201"  Part="1"
 F 0 "L201" H 6262 3138 60  0000 C CNN
 F 1 "IHLP2525CZER6R8M01" H 6262 3032 60  0000 C CNN
@@
 Wire Wire Line
 	6652 2850 7050 2850
+$Comp
+L SamacSys_Parts:SL08_10001 RT201
+U 1 1 626F9195
+P 2040 3650
+F 0 "RT201" H 2440 3915 50  0000 C CNN
+F 1 "SL08_10001" H 2440 3824 50  0000 C CNN
+F 2 "SamacSys_Parts:SL0810001" H 2690 3750 50  0001 L CNN
+F 3 "https://componentsearchengine.com/Datasheets/1/SL08 10001.pdf" H 2690 3650 50  0001 L CNN
+F 4 "NTC THERMISTOR; Product Range:SL08 Series; Disc Size:8mm; Zero Power Resistance at 25C:10ohm; Approvals:-; Maximum Energy Rating at 25C:8J; Maximum Steady State Current at 25C:1A; Dissipation Constant:9mW/C; No. of Pins:2 RoHS Compliant: Yes" H 2690 3550 50  0001 L CNN "Description"
+F 5 "19.3" H 2690 3450 50  0001 L CNN "Height"
+F 6 "995-SL0810001" H 2690 3350 50  0001 L CNN "Mouser Part Number"
+F 7 "https://www.mouser.com/Search/Refine.aspx?Keyword=995-SL0810001" H 2690 3250 50  0001 L CNN "Mouser Price/Stock"
+F 8 "AMETHERM" H 2690 3150 50  0001 L CNN "Manufacturer_Name"
+F 9 "SL08 10001" H 2690 3050 50  0001 L CNN "Manufacturer_Part_Number"
+	1    2040 3650
+	1    0    0    -1
+$EndComp
+$Comp
+L SamacSys_Parts:MF-MSMF050-2 F201
+U 1 1 626FB5FC
+P 1340 3650
+F 0 "F201" H 1690 3875 50  0000 C CNN
+F 1 "MF-MSMF050-2" H 1690 3784 50  0000 C CNN
+F 2 "SamacSys_Parts:FUSC4632X85N" H 1890 3700 50  0001 L CNN
+F 3 "https://www.bourns.com/pdfs/mfmsmf.pdf" H 1890 3600 50  0001 L CNN
+F 4 "Fuse, PTC, Resettable, SMD, 1812, 500mA Bourns 0.5A Surface Mount Resettable Fuse, 15 V" H 1890 3500 50  0001 L CNN "Description"
+F 5 "0.85" H 1890 3400 50  0001 L CNN "Height"
+F 6 "652-MF-MSMF050-2" H 1890 3300 50  0001 L CNN "Mouser Part Number"
+F 7 "https://www.mouser.co.uk/ProductDetail/Bourns/MF-MSMF050-2?qs=t3shhpq1i1DZ7OBD5kLNoA%3D%3D" H 1890 3200 50  0001 L CNN "Mouser Price/Stock"
+F 8 "Bourns" H 1890 3100 50  0001 L CNN "Manufacturer_Name"
+F 9 "MF-MSMF050-2" H 1890 3000 50  0001 L CNN "Manufacturer_Part_Number"
+	1    1340 3650
+	1    0    0    -1
+$EndComp
+Wire Wire Line
+	2840 3650 3210 3650
+Connection ~ 3210 3650
+Wire Notes Line
+	1470 3260 1470 3960
+Wire Notes Line
+	1470 3960 2790 3960
+Wire Notes Line
+	2790 3960 2790 3260
+Wire Notes Line
+	2790 3260 1470 3260
+Text Notes 1720 3190 0    50   ~ 0
+Current limiting circuit
 $EndSCHEMATC

Commit message: temp2
Parts:
- C201, C202: footprint Capacitor_SMD:C_1210_3225Metric -> Capacitor_SMD:C_1206_3216Metric
- C206, C208: footprint Capacitor_SMD:C_1210_3225Metric -> Capacitor_SMD:C_0805_2012Metric
Changed lines of the file:
@@
 F 0 "C206" H 6565 3296 50  0000 L CNN
 F 1 "47uF" H 6565 3205 50  0000 L CNN
-F 2 "Capacitor_SMD:C_1210_3225Metric" H 6488 3100 50  0001 C CNN
+F 2 "Capacitor_SMD:C_0805_2012Metric" H 6488 3100 50  0001 C CNN
 F 3 "~" H 6450 3250 50  0001 C CNN
 	1    6450 3250
@@
 F 0 "C208" H 7165 3296 50  0000 L CNN
 F 1 "47uF" H 7165 3205 50  0000 L CNN
-F 2 "Capacitor_SMD:C_1210_3225Metric" H 7088 3100 50  0001 C CNN
+F 2 "Capacitor_SMD:C_0805_2012Metric" H 7088 3100 50  0001 C CNN
 F 3 "~" H 7050 3250 50  0001 C CNN
 	1    7050 3250
@@
 F 0 "C202" H 4015 3846 50  0000 L CNN
 F 1 "22uf" H 4015 3755 50  0000 L CNN
-F 2 "Capacitor_SMD:C_1210_3225Metric" H 3938 3650 50  0001 C CNN
+F 2 "Capacitor_SMD:C_1206_3216Metric" H 3938 3650 50  0001 C CNN
 F 3 "~" H 3900 3800 50  0001 C CNN
 	1    3900 3800
@@
 F 0 "C201" H 3635 3846 50  0000 L CNN
 F 1 "22uf" H 3635 3755 50  0000 L CNN
-F 2 "Capacitor_SMD:C_1210_3225Metric" H 3558 3650 50  0001 C CNN
+F 2 "Capacitor_SMD:C_1206_3216Metric" H 3558 3650 50  0001 C CNN
 F 3 "~" H 3520 3800 50  0001 C CNN
 	1    3520 3800

Commit message: print
Parts:
- R201: value 56.2k -> 56k
- R202: value 10.2k -> 10k
- R203: value 1.78k -> 1.8k
Changed lines of the file:
@@
 AR Path="/61A31DC2/61A8D169" Ref="R201"  Part="1"
 F 0 "R201" H 5920 4346 50  0000 L CNN
-F 1 "56.2k" H 5920 4255 50  0000 L CNN
+F 1 "56k" H 5920 4255 50  0000 L CNN
 F 2 "Resistor_SMD:R_0805_2012Metric" V 5780 4300 50  0001 C CNN
 F 3 "~" H 5850 4300 50  0001 C CNN
@@
 AR Path="/61A31DC2/61A8D17A" Ref="R202"  Part="1"
 F 0 "R202" H 7470 3636 50  0000 L CNN
-F 1 "10.2k" H 7470 3545 50  0000 L CNN
+F 1 "10k" H 7470 3545 50  0000 L CNN
 F 2 "Resistor_SMD:R_0805_2012Metric" V 7330 3590 50  0001 C CNN
 F 3 "~" H 7400 3590 50  0001 C CNN
@@
 AR Path="/61A31DC2/61A8D180" Ref="R203"  Part="1"
 F 0 "R203" H 7470 4596 50  0000 L CNN
-F 1 "1.78k" H 7470 4505 50  0000 L CNN
+F 1 "1.8k" H 7470 4505 50  0000 L CNN
 F 2 "Resistor_SMD:R_0805_2012Metric" V 7330 4550 50  0001 C CNN
 F 3 "~" H 7400 4550 50  0001 C CNN
