File: CI_ComPCB/Transmiter.sch (KiCad schematic (older format))
At the start: 7 parts, among them J501 RJ45_LED_Shielded, J502 RJ45_LED_Shielded

Commit message: Sensor_SplitterPrint
Parts:
- Converter501, Converter502: symbol CI_ComPCB-rescue:TxRx-RS485-New_Library-RackComm-rescue-CI_ComPCB-rescue -> CI_ComPCB-rescue:TxRx-RS485-New_Library-RackComm-rescue-CI_ComPCB-rescue-CI_ComPCB-rescue
- D501: symbol CI_ComPCB-rescue:SS34-SamacSys_Parts -> CI_ComPCB-rescue:SS34-SamacSys_Parts-CI_ComPCB-rescue
Changed lines of the file:
@@
 $EndDescr
 $Comp
-L CI_ComPCB-rescue:TxRx-RS485-New_Library-RackComm-rescue-CI_ComPCB-rescue Converter?
+L CI_ComPCB-rescue:TxRx-RS485-New_Library-RackComm-rescue-CI_ComPCB-rescue-CI_ComPCB-rescue Converter?
 U 1 1 61AB1847
 P 3930 4500
@@
 $EndComp
 $Comp
-L CI_ComPCB-rescue:TxRx-RS485-New_Library-RackComm-rescue-CI_ComPCB-rescue Converter?
+L CI_ComPCB-rescue:TxRx-RS485-New_Library-RackComm-rescue-CI_ComPCB-rescue-CI_ComPCB-rescue Converter?
 U 1 1 61AB184D
 P 3930 5080
@@
 	6020 4990 6810 4990
 $Comp
-L CI_ComPCB-rescue:SS34-SamacSys_Parts D?
+L CI_ComPCB-rescue:SS34-SamacSys_Parts-CI_ComPCB-rescue D?
 U 1 1 614B2CBA
 P 6340 4780
