File: CI_ComPCB/Relay_Switches.sch (KiCad schematic (older format))
At the start: 22 parts, among them J601 Conn_01x02_Male, J602 Conn_01x02_Male, J603 Conn_01x03_Male, J604 Conn_01x03_Male, J605 Conn_01x02_Male, K601 SRD-05VDC-SL-C, K602 SRD-05VDC-SL-C, Q601 2N3904, Q602 2N3904

Commit message: Sensor_SplitterPrint
Parts:
- D601, D602, D606: symbol CI_ComPCB-rescue:LTST-C190GKT-dk_LED-Indication-Discrete -> CI_ComPCB-rescue:LTST-C190GKT-dk_LED-Indication-Discrete-CI_ComPCB-rescue
- D605: symbol CI_ComPCB-rescue:SS34-SamacSys_Parts -> CI_ComPCB-rescue:SS34-SamacSys_Parts-CI_ComPCB-rescue
- K601, K602: symbol SRD-05VDC-SL-C:SRD-05VDC-SL-C -> CI_ComPCB-rescue:SRD-05VDC-SL-C-SRD-05VDC-SL-C
Changed lines of the file:
@@
 $EndComp
 $Comp
-L CI_ComPCB-rescue:LTST-C190GKT-dk_LED-Indication-Discrete D?
+L CI_ComPCB-rescue:LTST-C190GKT-dk_LED-Indication-Discrete-CI_ComPCB-rescue D?
 U 1 1 6173F3C7
 P 5000 2600
@@
 $EndComp
 $Comp
-L CI_ComPCB-rescue:LTST-C190GKT-dk_LED-Indication-Discrete D?
+L CI_ComPCB-rescue:LTST-C190GKT-dk_LED-Indication-Discrete-CI_ComPCB-rescue D?
 U 1 1 617D35BE
 P 5050 5050
@@
 $EndComp
 $Comp
-L CI_ComPCB-rescue:LTST-C190GKT-dk_LED-Indication-Discrete D?
+L CI_ComPCB-rescue:LTST-C190GKT-dk_LED-Indication-Discrete-CI_ComPCB-rescue D?
 U 1 1 617E89E6
 P 8414 4500
@@
 EPower
 $Comp
-L CI_ComPCB-rescue:SS34-SamacSys_Parts D?
+L CI_ComPCB-rescue:SS34-SamacSys_Parts-CI_ComPCB-rescue D?
 U 1 1 617E89F3
 P 7260 5000
@@
 $EndComp
 $Comp
-L SRD-05VDC-SL-C:SRD-05VDC-SL-C K601
+L CI_ComPCB-rescue:SRD-05VDC-SL-C-SRD-05VDC-SL-C K601
 U 1 1 6188DFD6
 P 6600 2448
@@
 	7048 2148 7048 2444
 $Comp
-L SRD-05VDC-SL-C:SRD-05VDC-SL-C K602
+L CI_ComPCB-rescue:SRD-05VDC-SL-C-SRD-05VDC-SL-C K602
 U 1 1 617EEB4B
 P 6650 4900
