File: CI_ComPCB/Max 485 transmitter/Max 485 transmitter.kicad_pcb (KiCad board)
At the start: 2 copper layers, 37.5 x 15.9 mm, 23 parts, among them IC101 74HC04D,653, IC102 SP485EEN-L_TR, J101 Conn_01x04_Male, J102 Conn_01x03_Male

Commit message: Transmitter print
Parts:
- removed J101: Conn_01x04_Male, Connector_PinHeader_2.54mm:PinHeader_1x04_P2.54mm_Vertical
- removed J102: Conn_01x03_Male, Connector_PinHeader_2.54mm:PinHeader_1x03_P2.54mm_Vertical
- added Converter101: TxRx-RS485-New_Library-RackComm-rescue-CI_ComPCB-rescue, CI_ComPCB:TXRX-AB, F.Cu at (103.2, 47.8)
- moved D103 0.16 mm to (129.3, 59.4)
Routing:
- net TX: track 26.2 -> 32.7 mm
- net 3v3: track 49.0 -> 54.9 mm
- net Comm: track 7.91 -> 13.0 mm
- net A: track 6.33 -> 11.2 mm
- net GND: track 37.0 -> 41.8 mm
- net B: track 5.86 -> 9.90 mm
- net RX: track 6.98 -> 8.23 mm
- net Net-(D103-Pad2): track 27.8 -> 26.8 mm
- net Net-(D103-Pad1): track 35.6 -> 36.2 mm
Other:
- board size 37.5 x 15.9 mm -> 43.2 x 15.9 mm

Commit message: switch
Parts:
- moved R1 5.44 mm to (127.8, 54.0)
- moved R3 4.68 mm to (107.3, 50.7)
- moved R0 4.45 mm to (141.6, 54.5)
- moved R9 4.45 mm to (141.6, 50.3)
- moved R4 3.90 mm to (109.9, 50.7)
- moved R5 3.85 mm to (112.4, 50.7)
- moved IC101 3.42 mm to (110.0, 57.1)
- moved R7 2.65 mm to (115.7, 50.2), turned to 0 degrees
- moved D1 2.38 mm to (116.2, 57.4)
- moved C1 2.22 mm to (118.4, 53.3)
- moved R8 2.11 mm to (118.7, 50.2), turned to 0 degrees
- moved C2 2.01 mm to (116.5, 61.6)
- moved D102 1.97 mm to (123.9, 49.5)
- moved D104 1.91 mm to (136.4, 57.7)
- moved D105 1.91 mm to (136.4, 61.3)
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Routing:
- net 3v3: track 54.9 -> 32.9 mm, vias 2 -> 0
- net GND: track 41.8 -> 53.2 mm, vias 5 -> 4
- net TX: track 32.7 -> 37.8 mm
- net Net-(D103-Pad2): track 26.8 -> 22.0 mm
- net Net-(D103-Pad1): track 36.2 -> 31.6 mm
- net Net-(IC101-Pad9): track 21.4 -> 24.8 mm
- net RX: track 8.23 -> 5.17 mm
- net Comm: track 13.0 -> 10.1 mm
- net Net-(IC101-Pad6): track 12.4 -> 15.2 mm
- net Net-(IC101-Pad12): track 7.38 -> 9.96 mm
- net Net-(D1-Pad1): track 14.1 -> 16.6 mm
- net Net-(D102-Pad2): track 4.74 -> 7.26 mm
- net Net-(C2-Pad1): track 24.6 -> 26.9 mm, vias 2 -> 0
- net Net-(D101-Pad2): track 3.30 -> 4.99 mm
- net A: track 11.2 -> 10.5 mm
Other:
- board size 43.2 x 15.9 mm -> 43.2 x 25.4 mm
- rule trace_min: 0.2 -> 0.1

Commit message: transmitter update
Parts:
- C1, C2: footprint Capacitor_SMD:C_0201_0603Metric -> Capacitor_SMD:C_0402_1005Metric
Routing:
- net GND: track 53.2 -> 48.8 mm

Commit message: converters debug
Other:
- board size 43.2 x 25.4 mm -> 43.2 x 16.5 mm
- rule trace_min: 0.1 -> 0.2
- board text added: "V1.0"
Changed lines of the file:
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@@
   (general
     (thickness 1.6)
-    (drawings 16)
+    (drawings 10)
     (tracks 203)
     (zones 0)
@@
     (zone_clearance 0.508)
     (zone_45_only no)
-    (trace_min 0.1)
+    (trace_min 0.2)
     (via_size 0.8)
     (via_drill 0.4)
@@
       (effects (font (size 1 1) (thickness 0.15)))
     )
-    (fp_text user %R (at 0 0) (layer F.Fab)
-      (effects (font (size 0.25 0.25) (thickness 0.04)))
-    )
     (fp_line (start -0.5 0.25) (end -0.5 -0.25) (layer F.Fab) (width 0.1))
     (fp_line (start -0.5 -0.25) (end 0.5 -0.25) (layer F.Fab) (width 0.1))
@@
     (fp_line (start 0.91 -0.46) (end 0.91 0.46) (layer F.CrtYd) (width 0.05))
     (fp_line (start 0.91 0.46) (end -0.91 0.46) (layer F.CrtYd) (width 0.05))
+    (fp_text user %R (at 0 0) (layer F.Fab)
+      (effects (font (size 0.25 0.25) (thickness 0.04)))
+    )
     (pad 2 smd roundrect (at 0.48 0) (size 0.56 0.62) (layers F.Cu F.Paste F.Mask) (roundrect_rratio 0.25)
       (net 1 GND))
@@
     (fp_text value 0.1u (at 0 1.16) (layer F.Fab)
       (effects (font (size 1 1) (thickness 0.15)))
-    )
-    (fp_text user %R (at 0 0) (layer F.Fab)
-      (effects (font (size 0.25 0.25) (thickness 0.04)))
     )
     (fp_line (start -0.5 0.25) (end -0.5 -0.25) (layer F.Fab) (width 0.1))
@@
     (fp_line (start 0.91 -0.46) (end 0.91 0.46) (layer F.CrtYd) (width 0.05))
     (fp_line (start 0.91 0.46) (end -0.91 0.46) (layer F.CrtYd) (width 0.05))
+    (fp_text user %R (at 0 0) (layer F.Fab)
+      (effects (font (size 0.25 0.25) (thickness 0.04)))
+    )
     (pad 2 smd roundrect (at 0.48 0) (size 0.56 0.62) (layers F.Cu F.Paste F.Mask) (roundrect_rratio 0.25)
       (net 1 GND))
@@
     )
   )
-  (gr_line (start 142.24 46.99) (end 127 46.99) (layer Edge.Cuts) (width 0.05))
-  (gr_line (start 127 44.45) (end 142.24 44.45) (layer Edge.Cuts) (width 0.05))
-  (gr_line (start 121.285 44.45) (end 102.87 44.45) (layer Edge.Cuts) (width 0.05))
-  (gr_line (start 102.87 46.99) (end 121.285 46.99) (layer Edge.Cuts) (width 0.05))
-  (gr_line (start 127 46.99) (end 127 44.45) (layer Edge.Cuts) (width 0.05))
-  (gr_line (start 121.285 44.45) (end 121.285 46.99) (layer Edge.Cuts) (width 0.05))
-  (gr_line (start 142.24 46.99) (end 146.05 46.99) (layer Edge.Cuts) (width 0.05))
-  (gr_line (start 142.24 44.45) (end 146.05 44.45) (layer Edge.Cuts) (width 0.05))
-  (gr_line (start 146.05 44.45) (end 146.05 38.1) (layer Edge.Cuts) (width 0.05))
-  (gr_line (start 102.87 38.1) (end 146.05 38.1) (layer Edge.Cuts) (width 0.05))
-  (gr_line (start 102.87 44.45) (end 102.87 38.1) (layer Edge.Cuts) (width 0.05))
   (gr_line (start 146.05 63.5) (end 146.05 46.99) (layer Edge.Cuts) (width 0.05))
   (gr_line (start 102.87 63.5) (end 146.05 63.5) (layer Edge.Cuts) (width 0.05))
+  (gr_line (start 102.87 46.99) (end 121.285 46.99) (layer Edge.Cuts) (width 0.05))
   (gr_line (start 102.87 46.99) (end 102.87 63.5) (layer Edge.Cuts) (width 0.05))
+  (gr_line (start 142.24 46.99) (end 146.05 46.99) (layer Edge.Cuts) (width 0.05))
+  (gr_line (start 142.24 46.99) (end 127 46.99) (layer Edge.Cuts) (width 0.05))
+  (gr_line (start 121.285 46.99) (end 127 46.99) (layer Edge.Cuts) (width 0.05))
+  (gr_text V1.0 (at 143.51 62.23) (layer F.SilkS)
+    (effects (font (size 1 1) (thickness 0.15)))
+  )
   (gr_text RX (at 127.6604 52.07) (layer F.SilkS)
     (effects (font (size 1.5 1.5) (thickness 0.3)))
